File: Projet pedaledisto/Projet pedaledisto.kicad_sch (KiCad schematic)
At the start: 18 parts

Commit message: Add files via upload
Parts:
- removed U?: TL081, symbol Amplifier_Operational:TL081
- added H1, H2, H3, H4: MountingHole_Pad, MountingHole:MountingHole_3.2mm_M3_Pad_Via, symbol Mechanical:MountingHole_Pad
- added J1, J2, J3: Conn_01x02, Connector_JST:JST_XH_B2B-XH-A_1x02_P2.50mm_Vertical, symbol Connector_Generic:Conn_01x02
- added R1: 50k, Resistor_SMD:R_0603_1608Metric_Pad0.98x0.95mm_HandSolder, symbol Device:R
- added R9: 5k, Resistor_SMD:R_0603_1608Metric_Pad0.98x0.95mm_HandSolder, symbol Device:R
- added U1: TL081, Package_SO:SOIC-8-1EP_3.9x4.9mm_P1.27mm_EP2.29x3mm, symbol Amplifier_Operational:TL081
- C1, C2, C3: footprint (none) -> Capacitor_SMD:C_0603_1608Metric_Pad1.08x0.95mm_HandSolder
- C4: renamed from C6; footprint (none) -> Capacitor_SMD:C_0603_1608Metric_Pad1.08x0.95mm_HandSolder
- C5: renamed from C4; footprint (none) -> Capacitor_SMD:C_0603_1608Metric_Pad1.08x0.95mm_HandSolder
- C6: renamed from C5; footprint (none) -> Capacitor_SMD:C_0603_1608Metric_Pad1.08x0.95mm_HandSolder
- D1, D2: footprint Diode_THT:D_DO-35_SOD27_P7.62mm_Horizontal -> Diode_SMD:D_0603_1608Metric_Pad1.05x0.95mm_HandSolder
- R2: renamed from R3; footprint (none) -> Resistor_SMD:R_0603_1608Metric_Pad0.98x0.95mm_HandSolder
- R3: renamed from R1; footprint (none) -> Resistor_SMD:R_0603_1608Metric_Pad0.98x0.95mm_HandSolder
- R4: renamed from R2; footprint (none) -> Resistor_SMD:R_0603_1608Metric_Pad0.98x0.95mm_HandSolder
- R5: renamed from R4; footprint (none) -> Resistor_SMD:R_0603_1608Metric_Pad0.98x0.95mm_HandSolder
- R6, R7: footprint (none) -> Resistor_SMD:R_0603_1608Metric_Pad0.98x0.95mm_HandSolder
- R8: renamed from R5; footprint (none) -> Resistor_SMD:R_0603_1608Metric_Pad0.98x0.95mm_HandSolder
- RV1: value 500K-reverse-log (C500K) -> 500K-lin(500k); footprint (none) -> Connector_JST:JST_XH_B3B-XH-A_1x03_P2.50mm_Vertical
- RV2: value 50K-log (A50K) -> 50K-lin(50K); footprint (none) -> Connector_JST:JST_XH_B3B-XH-A_1x03_P2.50mm_Vertical
Connections:
- net +9V: now also J1.2 (Pin_2), U1.7 (V+)
- net GND: now also H1.1, H2.1, H3.1, H4.1, J1.1 (Pin_1), J2.1 (Pin_1), J3.1 (Pin_1), R1.1, R9.1, U1.4 (V-)
- net Input: now reaches C1.1, C2.1
- net Input: now also J2.2 (Pin_2)
- net at R2.1, RV1.3: now also R1.2
- net at C5.1, R5.2: now also U1.6
- net at C3.2, R5.1: now also U1.2 (-)
- net at R3.2, R4.1: now also U1.3 (+)
- net Output: now reaches RV2.2
- net Output: now also J3.2 (Pin_2), R9.2
- no-connect marks 0 -> 2
Other:
- note added: "Power Input : +9V DC"
- note added: "Signal Input"
- note added: "Signal Output"
